File: hardware/co_sensor.kicad_pcb (KiCad board)
At the start: 2 copper layers, 80 x 40 mm, 43 parts, among them J1 Barrel_Jack, U1 NodeMCU1.0(ESP-12E), U2 MQ-7, U3 LM393ADR

Commit message: Adds gerber file and updates schematic to include hardware in BOM
Parts:
- J1: value Barrel_Jack -> PJ1-022-SMT-TR; footprint Connector_BarrelJack:BarrelJack_CUI_PJ-036AH-SMT_Horizontal -> PJ1-022-SMT:CUI_PJ1-022-SMT-TR
- moved J1 5.00 mm to (127.5, 122.5), turned to 0 degrees
Connections:
- J1 pad 3: (no net) -> Net-(J1-Pad3)
Routing:
- net VCC: track 121.0 -> 130.5 mm
Changed lines of the file:
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@@
     (thickness 1.6002)
     (drawings 12)
-    (tracks 63)
+    (tracks 67)
     (zones 0)
     (modules 43)
-    (nets 37)
+    (nets 38)
   )
   (page A3)
@@
     (visible_elements 7FFFFFFF)
     (pcbplotparams
-      (layerselection 0x00030_80000001)
+      (layerselection 0x01030_ffffffff)
       (usegerberextensions true)
       (usegerberattributes false)
@@
       (outputformat 1)
       (mirror false)
-      (drillshape 1)
+      (drillshape 0)
       (scaleselection 1)
       (outputdirectory ""))
@@
   (net 35 "Net-(U3-Pad6)")
   (net 36 "Net-(U3-Pad5)")
+  (net 37 "Net-(J1-Pad3)")
   (net_class Default "To jest domyślna klasa połączeń."
     (clearance 0.254)
@@
     (add_net GND)
     (add_net "Net-(D1-Pad2)")
+    (add_net "Net-(J1-Pad3)")
     (add_net "Net-(R1-Pad1)")
     (add_net "Net-(R2-Pad1)")
@@
     (add_net "Net-(U3-Pad7)")
     (add_net VCC)
+  )
+  (module PJ1-022-SMT:CUI_PJ1-022-SMT-TR (layer F.Cu)
+    (at 127.5 122.5)
+    (fp_text reference J1 (at -2.807305 -3.768105) (layer F.SilkS)
+      (effects (font (size 1.000827 1.000827) (thickness 0.015)))
+    )
+    (fp_text value PJ1-022-SMT-TR (at 5.42 3.685) (layer F.Fab)
+      (effects (font (size 1 1) (thickness 0.015)))
+    )
+    (fp_line (start 7.25 1.5) (end 6.25 1.5) (layer F.CrtYd) (width 0.05))
+    (fp_line (start 7.25 -1.5) (end 7.25 1.5) (layer F.CrtYd) (width 0.05))
+    (fp_line (start 6.25 -1.5) (end 7.25 -1.5) (layer F.CrtYd) (width 0.05))
+    (fp_line (start 0.95 5.1) (end 0.95 2.75) (layer F.CrtYd) (width 0.05))
+    (fp_line (start 5.05 5.1) (end 0.95 5.1) (layer F.CrtYd) (width 0.05))
+    (fp_line (start 5.05 2.75) (end 5.05 5.1) (layer F.CrtYd) (width 0.05))
+    (fp_line (start 6.05 -5.1) (end 6.05 -2.75) (layer F.CrtYd) (width 0.05))
+    (fp_line (start 1.95 -5.1) (end 6.05 -5.1) (layer F.CrtYd) (width 0.05))
+    (fp_line (start 1.95 -2.75) (end 1.95 -5.1) (layer F.CrtYd) (width 0.05))
+    (fp_line (start 5 2.5) (end 6 2.5) (layer F.SilkS) (width 0.127))
+    (fp_line (start 6 1.5) (end 6 2.5) (layer F.SilkS) (width 0.127))
+    (fp_line (start 6 -2.25) (end 6 -1.5) (layer F.SilkS) (width 0.127))
+    (fp_line (start 1.95 -2.75) (end -6.25 -2.75) (layer F.CrtYd) (width 0.05))
+    (fp_line (start 6.25 -2.75) (end 6.05 -2.75) (layer F.CrtYd) (width 0.05))
+    (fp_line (start 6.25 -1.5) (end 6.25 -2.75) (layer F.CrtYd) (width 0.05))
+    (fp_line (start 6.25 2.75) (end 6.25 1.5) (layer F.CrtYd) (width 0.05))
+    (fp_line (start 5.05 2.75) (end 6.25 2.75) (layer F.CrtYd) (width 0.05))
+    (fp_line (start -6.25 2.75) (end 0.95 2.75) (layer F.CrtYd) (width 0.05))
+    (fp_line (start -6.25 -2.75) (end -6.25 2.75) (layer F.CrtYd) (width 0.05))
+    (fp_line (start 2 -2.5) (end -6 -2.5) (layer F.SilkS) (width 0.127))
+    (fp_line (start -6 2.5) (end 0.75 2.5) (layer F.SilkS) (width 0.127))
+    (fp_line (start -6 -2.5) (end -6 2.5) (layer F.SilkS) (width 0.127))
+    (fp_line (start 6 -2.5) (end -6 -2.5) (layer F.Fab) (width 0.127))
+    (fp_line (start 6 2.5) (end 6 -2.5) (layer F.Fab) (width 0.127))
+    (fp_line (start -6 2.5) (end 6 2.5) (layer F.Fab) (width 0.127))
+    (fp_line (start -6 -2.5) (end -6 2.5) (layer F.Fab) (width 0.127))
+    (fp_circle (center 7.8 0.01) (end 8 0.01) (layer F.SilkS) (width 0.4))
+    (pad None np_thru_hole circle (at -3 0) (size 1.6 1.6) (drill 1.6) (layers *.Cu *.Mask))
+    (pad None np_thru_hole circle (at 2.5 0) (size 1.6 1.6) (drill 1.6) (layers *.Cu *.Mask))
+    (pad 2 smd rect (at 3 3.65) (size 3.5 2.3) (layers F.Cu F.Paste F.Mask)
+      (net 27 GND))
+    (pad 3 smd rect (at 4 -3.65) (size 3.5 2.3) (layers F.Cu F.Paste F.Mask)
+      (net 37 "Net-(J1-Pad3)"))
+    (pad 1 smd rect (at 6 0) (size 2 2.5) (layers F.Cu F.Paste F.Mask)
+      (net 26 VCC))
+    (model /home/vmoeykens/projects/kicad-libraries/PJ1-022-SMT-TR/CUI_DEVICES_PJ1-022-SMT-TR.step
+      (offset (xyz -5.9944 0 0))
+      (scale (xyz 1 1 1))
+      (rotate (xyz -90 0 90))
+    )
   )
   (module Symbol:OSHW-Logo2_9.8x8mm_Copper (layer B.Cu)
@@
       (net 27 GND) (zone_connect 2))
   )
-  (module Connector_BarrelJack:BarrelJack_CUI_PJ-036AH-SMT_Horizontal (layer F.Cu)
-    (at 132.5 122.5 270)
-    (descr "Surface-mount DC Barrel Jack, http://www.cui.com/product/resource/pj-036ah-smt.pdf")
-    (tags "Power Jack SMT")
-    (attr smd)
-    (fp_text reference J1 (at -4.5 -5.75 90) (layer F.SilkS)
-      (effects (font (size 1 1) (thickness 0.15)))
-    )
-    (fp_text value Barrel_Jack (at 0 11.25 90) (layer F.Fab)
-      (effects (font (size 1 1) (thickness 0.15)))
-    )
-    (fp_circle (center 0.7 -3.4) (end 0.75 -2.95) (layer F.Fab) (width 0.12))
-    (fp_line (start 4.1 -2.5) (end 4.1 -4.5) (layer F.Fab) (width 0.1))
-    (fp_line (start 4.5 -2.5) (end 4.1 -2.5) (layer F.Fab) (width 0.1))
-    (fp_line (start 4.5 10) (end 4.5 -2.5) (layer F.Fab) (width 0.1))
-    (fp_line (start -4.5 10) (end 4.5 10) (layer F.Fab) (width 0.1))
-    (fp_line (start -4.5 -2.5) (end -4.5 10) (layer F.Fab) (width 0.1))
-    (fp_line (start -4.1 -2.5) (end -4.5 -2.5) (layer F.Fab) (width 0.1))
-    (fp_line (start -4.1 -4.5) (end -4.1 -2.5) (layer F.Fab) (width 0.1))
-    (fp_line (start 4.1 -4.5) (end -4.1 -4.5) (layer F.Fab) (width 0.1))
-    (fp_line (start -1.19 -8.24) (end 0.55 -8.24) (layer F.SilkS) (width 0.12))
-    (fp_line (start -1.19 -6.5) (end -1.19 -8.24) (layer F.SilkS) (width 0.12))
-    (fp_line (start 4.6 -2.6) (end 4.6 -0.15) (layer F.SilkS) (width 0.12))
-    (fp_line (start 4.2 -2.6) (end 4.6 -2.6) (layer F.SilkS) (width 0.12))
-    (fp_line (start 4.2 -4.6) (end 4.2 -2.6) (layer F.SilkS) (width 0.12))
-    (fp_line (start 2.6 -4.6) (end 4.2 -4.6) (layer F.SilkS) (width 0.12))
-    (fp_line (start -4.2 -4.6) (end -1.2 -4.6) (layer F.SilkS) (width 0.12))
-    (fp_line (start -4.2 -2.6) (end -4.2 -4.6) (layer F.SilkS) (width 0.12))
-    (fp_line (start -4.6 -2.6) (end -4.2 -2.6) (layer F.SilkS) (width 0.12))
-    (fp_line (start -4.6 -0.15) (end -4.6 -2.6) (layer F.SilkS) (width 0.12))
-    (fp_line (start -4.6 10.1) (end -4.6 6.55) (layer F.SilkS) (width 0.12))
-    (fp_line (start 4.6 10.1) (end -4.6 10.1) (layer F.SilkS) (width 0.12))
-    (fp_line (start 4.6 6.55) (end 4.6 10.1) (layer F.SilkS) (width 0.12))
-    (fp_line (start 8.9 -8.5) (end -8.9 -8.5) (layer F.CrtYd) (width 0.05))
-    (fp_line (start 8.9 10.5) (end 8.9 -8.5) (layer F.CrtYd) (width 0.05))
-    (fp_line (start -8.9 10.5) (end 8.9 10.5) (layer F.CrtYd) (width 0.05))
-    (fp_line (start -8.9 -8.5) (end -8.9 10.5) (layer F.CrtYd) (width 0.05))
-    (fp_text user %R (at 0 0 90) (layer F.Fab)
-      (effects (font (size 1 1) (thickness 0.15)))
-    )
-    (pad "" np_thru_hole circle (at 0 7 270) (size 2 2) (drill 2) (layers *.Cu *.Mask))
-    (pad 3 smd rect (at 6.45 3.2 270) (size 3.9 6.2) (layers F.Cu F.Paste F.Mask))
-    (pad 2 smd rect (at -6.45 3.2 270) (size 3.9 6.2) (layers F.Cu F.Paste F.Mask)
-      (net 27 GND))
-    (pad 1 smd rect (at 0.7 -5.8 270) (size 3.3 4.4) (layers F.Cu F.Paste F.Mask)
-      (net 26 VCC))
-    (model ${KISYS3DMOD}/Connector_BarrelJack.3dshapes/BarrelJack_CUI_PJ-036AH-SMT_Horizontal.wrl
-      (at (xyz 0 0 0))
-      (scale (xyz 1 1 1))
-      (rotate (xyz 0 0 0))
-    )
-  )
   (module Resistor_SMD:R_0805_2012Metric (layer B.Cu)
     (at 147.44 120.22 180)
@@
   (segment (start 138.3 119.2) (end 138.3 123.2) (width 0.254) (layer F.Cu) (net 26))
   (segment (start 140 117.5) (end 138.3 119.2) (width 0.254) (layer F.Cu) (net 26))
+  (segment (start 139.371383 117.5) (end 140 117.5) (width 0.254) (layer F.Cu) (net 26))
+  (segment (start 133.5 120.996) (end 136.996 117.5) (width 0.254) (layer F.Cu) (net 26))
+  (segment (start 136.996 117.5) (end 139.371383 117.5) (width 0.254) (layer F.Cu) (net 26))
+  (segment (start 133.5 122.5) (end 133.5 120.996) (width 0.254) (layer F.Cu) (net 26))
   (segment (start 159.14 127.88) (end 151.13 135.89) (width 0.254) (layer F.Cu) (net 28))
   (segment (start 159.14 126.39) (end 159.14 127.88) (width 0.254) (layer F.Cu) (net 28))
@@
   (segment (start 148.47 124.03) (end 148.3775 124.03) (width 0.254) (layer B.Cu) (net 30))
   (segment (start 152.5 120) (end 148.47 124.03) (width 0.254) (layer B.Cu) (net 30))
+  (via (at 145 112.5) (size 0.889) (drill 0.635) (layers F.Cu B.Cu) (net 32))
+  (segment (start 145 110.225) (end 145 112.5) (width 0.254) (layer F.Cu) (net 32))
+  (segment (start 142.5 108.6) (end 143.375 108.6) (width 0.254) (layer F.Cu) (net 32))
+  (segment (start 143.375 108.6) (end 145 110.225) (width 0.254) (layer F.Cu) (net 32))
+  (segment (start 145 114.9075) (end 146.5025 116.41) (width 0.254) (layer B.Cu) (net 32))
+  (segment (start 145 112.5) (end 145 114.9075) (width 0.254) (layer B.Cu) (net 32))
   (via (at 150 130) (size 0.889) (drill 0.635) (layers F.Cu B.Cu) (net 33))
   (segment (start 148.4375 127.5) (end 148.4375 128.4375) (width 0.254) (layer B.Cu) (net 33))
@@
   (segment (start 142.5 122.5) (end 142.5 111.4) (width 0.254) (layer F.Cu) (net 33))
   (segment (start 150 130) (end 142.5 122.5) (width 0.254) (layer F.Cu) (net 33))
-  (via (at 145 112.5) (size 0.889) (drill 0.635) (layers F.Cu B.Cu) (net 32))
-  (segment (start 145 110.225) (end 145 112.5) (width 0.254) (layer F.Cu) (net 32))
-  (segment (start 142.5 108.6) (end 143.375 108.6) (width 0.254) (layer F.Cu) (net 32))
-  (segment (start 143.375 108.6) (end 145 110.225) (width 0.254) (layer F.Cu) (net 32))
-  (segment (start 145 114.9075) (end 146.5025 116.41) (width 0.254) (layer B.Cu) (net 32))
-  (segment (start 145 112.5) (end 145 114.9075) (width 0.254) (layer B.Cu) (net 32))
   (segment (start 147.35649 128.58101) (end 147.951973 127.985527) (width 0.254) (layer B.Cu) (net 33))
   (segment (start 139.9384 124.9638) (end 143.55561 128.58101) (width 0.254) (layer B.Cu) (net 33))
